File: pcb/PanelModular.kicad_pcb (KiCad board)
At the start: 2 copper layers, 158.8 x 68.8 mm, 45 parts, among them J1 KEY_1, J1.1 Conn_01x08, J10 KEY_10, J11 LED_1, J12 LED_2, J13 LED_3, J14 LED_4, J15 LED_5, J16 LED_6, J17 LED_7, J18 LED_8, J19 ADC_1, J2 KEY_2, J2.1 Conn_01x08, J20 ADC_2, J21 ADC_3, J22 E_STOP, J23 ENCODER, J24 START, J25 STOP, J26 E_STOP_LED, J27 WS2811, J28 MIST, J29 KEY_11, J3 KEY_3, J30 KEY_12, J31 BREAK, J4 KEY_4, J5 KEY_5, J6 KEY_6, J7 KEY_7, J8 KEY_8, J9 KEY_9, U1 LM7805_TO220, U2 Pico, U4 74LVC1G17

Commit message: I2C ready version
Parts:
- added J32: I2C_3V3, Connector_JST:JST_XH_B4B-XH-A_1x04_P2.50mm_Vertical, F.Cu at (173.4, 119.4)
- added J33: I2C_5V, Connector_JST:JST_XH_B4B-XH-A_1x04_P2.50mm_Vertical, F.Cu at (188.0, 119.4)
- added JP1: LED_Power_Jumper, Jumper:SolderJumper-3_P1.3mm_Bridged12_Pad1.0x1.5mm_NumberLabels, F.Cu at (167.6, 64.1)
- added JP2: I2C_Power Jumper, Jumper:SolderJumper-3_P1.3mm_Bridged12_Pad1.0x1.5mm_NumberLabels, F.Cu at (166.4, 121.9)
- added JP3: OverrideU4, Jumper:SolderJumper-2_P1.3mm_Open_Pad1.0x1.5mm, F.Cu at (92.1, 106.0)
- added JP4: Enable U4, Jumper:SolderJumper-2_P1.3mm_Bridged_Pad1.0x1.5mm, F.Cu at (100.3, 108.0)
- added Q1: BSS138, Package_TO_SOT_SMD:SOT-23, F.Cu at (185.1, 107.0)
- added Q2: BSS138, Package_TO_SOT_SMD:SOT-23, F.Cu at (194.0, 107.0)
- added R2: 10K, Resistor_SMD:R_0805_2012Metric_Pad1.20x1.40mm_HandSolder, F.Cu at (188.6, 105.8)
- added R3: 10K, Resistor_SMD:R_0805_2012Metric_Pad1.20x1.40mm_HandSolder, F.Cu at (185.2, 110.5)
- added R4: 10K, Resistor_SMD:R_0805_2012Metric_Pad1.20x1.40mm_HandSolder, F.Cu at (193.9, 110.5)
- added R5: 10K, Resistor_SMD:R_0805_2012Metric_Pad1.20x1.40mm_HandSolder, F.Cu at (197.5, 105.8)
- added U3: PCF8574, Package_SO:SO-16_5.3x10.2mm_P1.27mm, F.Cu at (185.4, 93.3)
- R1, U4: moved to F.Cu
- moved U4 0.32 mm to (96.4, 105.4), turned to 0 degrees
- moved R1 0.13 mm to (96.5, 108.6), turned to 180 degrees
Connections:
- net MIST_AIR_3V3 renamed MIST_AIR
- net MIST_VALVE_3V3 renamed MIST_VALVE
- net REMOTE_EN_3V3 renamed REMOTE_EN
- D1 pad 14: +24V -> +U_LED
- D2 pad 14: +24V -> +U_LED
- J11 pad 2: +24V -> +U_LED
- J12 pad 2: +24V -> +U_LED
- J13 pad 2: +24V -> +U_LED
- J14 pad 2: +24V -> +U_LED
- J15 pad 2: +24V -> +U_LED
- J16 pad 2: +24V -> +U_LED
- J17 pad 2: +24V -> +U_LED
- J18 pad 2: +24V -> +U_LED
- J28 pad 3: +12V -> +5V
- R1 pad 1: Net-(R1-Pad1) -> Net-(JP3-B)
- U2 pad 16: WS_DATA -> SDA
- U2 pad 17: unconnected-(U2-GPIO13-Pad17) -> SCL
- U2 pad 19: LED_8 -> SDA2
- U2 pad 20: LED_7 -> SCL2
- U2 pad 21: LED_6 -> unconnected-(U2-GPIO16-Pad21)
- U2 pad 22: LED_5 -> unconnected-(U2-GPIO17-Pad22)
- U2 pad 24: LED_1 -> unconnected-(U2-GPIO18-Pad24)
- U2 pad 25: LED_2 -> unconnected-(U2-GPIO19-Pad25)
- U2 pad 26: LED_3 -> unconnected-(U2-GPIO20-Pad26)
- U2 pad 27: LED_4 -> WS_DATA
- U4 pad 4: Net-(R1-Pad1) -> Net-(JP4-A)
Routing:
- net +U_LED: track 0.00 -> 178.6 mm, vias 0 -> 3
- net SDA: track 0.00 -> 152.0 mm
- net SCL: track 0.00 -> 151.0 mm
- net +24V: track 231.2 -> 90.6 mm, vias 0 -> 1
- net SDA2: track 0.00 -> 99.8 mm, vias 0 -> 1
- net +3.3V: track 110.8 -> 204.8 mm, vias 0 -> 2
- net +5V: track 237.6 -> 328.0 mm, vias 2 -> 4
- net SCL2: track 0.00 -> 88.0 mm, vias 0 -> 1
- net LED_8: track 92.8 -> 15.4 mm, vias 1 -> 0
- net LED_4: track 91.6 -> 21.9 mm
- net LED_7: track 87.7 -> 19.3 mm, vias 1 -> 0
- net LED_3: track 84.4 -> 18.8 mm
- net LED_2: track 78.9 -> 15.8 mm
- net LED_1: track 76.8 -> 16.5 mm
- net LED_5: track 80.1 -> 25.4 mm
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Other:
- board size 158.8 x 68.8 mm -> 160 x 69 mm
- board text added: "12V"
- board text added: "24V"
- board text added: "3.3V"
- board text added: "5V"
- board text added: "GND"
- board text added: "LED"

Commit message: The first ordered Version, missing i2c pullups and wrong i2c connected to external
Parts:
- added C3: C, Capacitor_SMD:C_0805_2012Metric_Pad1.18x1.45mm_HandSolder, F.Cu at (178.4, 89.9)
- added J34: Reserve, Connector_JST:JST_XH_B6B-XH-A_1x06_P2.50mm_Vertical, F.Cu at (55.2, 72.6)
- added J35: POW_KEY_MAN, Connector_JST:JST_XH_B2B-XH-A_1x02_P2.50mm_Vertical, F.Cu at (125.7, 94.6)
- added Q3: BSS138, Package_TO_SOT_SMD:SOT-23_Handsoldering, F.Cu at (82.5, 105.7)
- added R6: 10K, Resistor_SMD:R_0805_2012Metric_Pad1.20x1.40mm_HandSolder, F.Cu at (78.0, 107.2)
- added R7: 10K, Resistor_SMD:R_0805_2012Metric_Pad1.20x1.40mm_HandSolder, F.Cu at (197.3, 101.2)
- added R8: 10K, Resistor_SMD:R_0805_2012Metric_Pad1.20x1.40mm_HandSolder, F.Cu at (197.3, 99.1)
- J23: value ENCODER -> POWER_KEY; footprint Connector_JST:JST_XH_B6B-XH-A_1x06_P2.50mm_Vertical -> Connector_JST:JST_XH_B2B-XH-A_1x02_P2.50mm_Vertical
- Q1, Q2: footprint Package_TO_SOT_SMD:SOT-23 -> Package_TO_SOT_SMD:SOT-23_Handsoldering
- U3: footprint Package_SO:SO-16_5.3x10.2mm_P1.27mm -> Library:SO-16_7,7x10.2mm_P1.27mm-PCF8574
- moved J1.1 34.0 mm to (63.7, 64.8), turned to 0 degrees
- moved J2.1 34.0 mm to (63.7, 81.3), turned to 0 degrees
- moved J28 2.16 mm to (108.6, 69.8)
- moved U3 1.92 mm to (185.4, 95.2)
- moved R2 0.89 mm to (189.5, 105.8)
- moved R5 0.89 mm to (198.4, 105.8)
- moved JP4 0.51 mm to (100.8, 108.0)
- moved R1 0.38 mm to (96.5, 109.0)
Connections:
- J2.1 pad 4: ENCODER_A+ -> POWER_EN
- J2.1 pad 5: ENCODER_A- -> RESERVE1
- J2.1 pad 6: ENCODER_B+ -> RESERVE2
- J2.1 pad 7: ENCODER_B- -> RESERVE3
- J23 pad 2: +5V -> POWER_KEY
- J32 pad 2: SDA -> SDA2
- J32 pad 3: SCL -> SCL2
- U2 pad 25: unconnected-(U2-GPIO19-Pad25) -> POWER_EN_3V3
- U2 pad 26: unconnected-(U2-GPIO20-Pad26) -> POWER_KEY
- U3 pad 14: SDA -> SCL
- U3 pad 15: SCL -> SDA
Routing:
- net SDA: track 152.0 -> 1.35 mm
- net SCL: track 151.0 -> 0.65 mm
- net POWER_EN: track 0.00 -> 127.8 mm, vias 0 -> 1
- net ENCODER_B-: track 72.7 -> 0.00 mm
- net ENCODER_B+: track 65.1 -> 0.00 mm
- net ENCODER_A-: track 56.8 -> 0.00 mm
- net ENCODER_A+: track 48.9 -> 0.00 mm
- net RESERVE3: track 0.00 -> 48.4 mm
- net RESERVE2: track 0.00 -> 44.9 mm
- net STOP_KEY: track 86.8 -> 45.1 mm
- net RESERVE1: track 0.00 -> 41.6 mm
- net +12V: track 104.2 -> 143.9 mm, vias 2 -> 0
- net BREAK_KEY: track 67.4 -> 29.0 mm
- net +24V: track 90.6 -> 129.0 mm
- net POWER_KEY: track 0.00 -> 29.1 mm
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
Commit message: Revert "The first ordered Version, missing i2c pullups and wrong i2c connected to external"
This reverts commit 4b4ee199a77fa0146eabba4f0e18928ce2f89e34.
Parts:
- removed C3: C, Capacitor_SMD:C_0805_2012Metric_Pad1.18x1.45mm_HandSolder
- removed J34: Reserve, Connector_JST:JST_XH_B6B-XH-A_1x06_P2.50mm_Vertical
- removed J35: POW_KEY_MAN, Connector_JST:JST_XH_B2B-XH-A_1x02_P2.50mm_Vertical
- removed Q3: BSS138, Package_TO_SOT_SMD:SOT-23_Handsoldering
- removed R6, R7, R8: 10K, Resistor_SMD:R_0805_2012Metric_Pad1.20x1.40mm_HandSolder
- J23: value POWER_KEY -> ENCODER; footprint Connector_JST:JST_XH_B2B-XH-A_1x02_P2.50mm_Vertical -> Connector_JST:JST_XH_B6B-XH-A_1x06_P2.50mm_Vertical
- Q1, Q2: footprint Package_TO_SOT_SMD:SOT-23_Handsoldering -> Package_TO_SOT_SMD:SOT-23
- U3: footprint Library:SO-16_7,7x10.2mm_P1.27mm-PCF8574 -> Package_SO:SO-16_5.3x10.2mm_P1.27mm
- moved J1.1 34.0 mm to (97.5, 68.6), turned to 180 degrees
- moved J2.1 34.0 mm to (97.5, 85.6), turned to 180 degrees
- moved J28 2.16 mm to (107.3, 68.1)
- moved U3 1.92 mm to (185.4, 93.3)
- moved R2 0.89 mm to (188.6, 105.8)
- moved R5 0.89 mm to (197.5, 105.8)
- moved JP4 0.51 mm to (100.3, 108.0)
- moved R1 0.38 mm to (96.5, 108.6)
Connections:
- J2.1 pad 4: POWER_EN -> ENCODER_A+
- J2.1 pad 5: RESERVE1 -> ENCODER_A-
- J2.1 pad 6: RESERVE2 -> ENCODER_B+
- J2.1 pad 7: RESERVE3 -> ENCODER_B-
- J23 pad 2: POWER_KEY -> +5V
- J32 pad 2: SDA2 -> SDA
- J32 pad 3: SCL2 -> SCL
- U2 pad 25: POWER_EN_3V3 -> unconnected-(U2-GPIO19-Pad25)
- U2 pad 26: POWER_KEY -> unconnected-(U2-GPIO20-Pad26)
- U3 pad 14: SCL -> SDA
- U3 pad 15: SDA -> SCL
Routing:
- net SDA: track 1.35 -> 152.0 mm
- net SCL: track 0.65 -> 151.0 mm
- net POWER_EN: track 127.8 -> 0.00 mm, vias 1 -> 0
- net ENCODER_B-: track 0.00 -> 72.7 mm
- net ENCODER_B+: track 0.00 -> 65.1 mm
- net ENCODER_A-: track 0.00 -> 56.8 mm
- net ENCODER_A+: track 0.00 -> 48.9 mm
- net RESERVE3: track 48.4 -> 0.00 mm
- net RESERVE2: track 44.9 -> 0.00 mm
- net STOP_KEY: track 45.1 -> 86.8 mm
- net RESERVE1: track 41.6 -> 0.00 mm
- net +12V: track 143.9 -> 104.2 mm, vias 0 -> 2
- net BREAK_KEY: track 29.0 -> 67.4 mm
- net +24V: track 129.0 -> 90.6 mm
- net POWER_KEY: track 29.1 -> 0.00 mm
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
Commit message: Really the first ordered Version, missing i2c pullups and wrong i2c connected to external
Parts:
- added C3: C, Capacitor_SMD:C_0805_2012Metric_Pad1.18x1.45mm_HandSolder, F.Cu at (178.4, 89.9)
- added J34: Reserve, Connector_JST:JST_XH_B6B-XH-A_1x06_P2.50mm_Vertical, F.Cu at (55.2, 72.6)
- added J35: POW_KEY_MAN, Connector_JST:JST_XH_B2B-XH-A_1x02_P2.50mm_Vertical, F.Cu at (125.7, 94.6)
- added Q3: BSS138, Package_TO_SOT_SMD:SOT-23_Handsoldering, F.Cu at (82.5, 105.7)
- added R6: 10K, Resistor_SMD:R_0805_2012Metric_Pad1.20x1.40mm_HandSolder, F.Cu at (78.0, 107.2)
- J23: value ENCODER -> POWER_KEY; footprint Connector_JST:JST_XH_B6B-XH-A_1x06_P2.50mm_Vertical -> Connector_JST:JST_XH_B2B-XH-A_1x02_P2.50mm_Vertical
- Q1, Q2: footprint Package_TO_SOT_SMD:SOT-23 -> Package_TO_SOT_SMD:SOT-23_Handsoldering
- U3: footprint Package_SO:SO-16_5.3x10.2mm_P1.27mm -> Library:SO-16_7,7x10.2mm_P1.27mm-PCF8574
- moved J1.1 34.0 mm to (63.7, 64.8), turned to 0 degrees
- moved J2.1 34.0 mm to (63.7, 81.3), turned to 0 degrees
- moved J28 2.16 mm to (108.6, 69.8)
- moved U3 1.92 mm to (185.4, 95.2)
- moved R2 0.89 mm to (189.5, 105.8)
- moved R5 0.89 mm to (198.4, 105.8)
- moved JP4 0.51 mm to (100.8, 108.0)
- moved R1 0.38 mm to (96.5, 109.0)
Connections:
- J2.1 pad 4: ENCODER_A+ -> POWER_EN
- J2.1 pad 5: ENCODER_A- -> RESERVE1
- J2.1 pad 6: ENCODER_B+ -> RESERVE2
- J2.1 pad 7: ENCODER_B- -> RESERVE3
- J23 pad 2: +5V -> POWER_KEY
- U2 pad 25: unconnected-(U2-GPIO19-Pad25) -> POWER_EN_3V3
- U2 pad 26: unconnected-(U2-GPIO20-Pad26) -> POWER_KEY
- U3 pad 14: SDA -> SCL
- U3 pad 15: SCL -> SDA
Routing:
- net POWER_EN: track 0.00 -> 127.8 mm, vias 0 -> 1
- net ENCODER_B-: track 72.7 -> 0.00 mm
- net ENCODER_B+: track 65.1 -> 0.00 mm
- net ENCODER_A-: track 56.8 -> 0.00 mm
- net ENCODER_A+: track 48.9 -> 0.00 mm
- net RESERVE3: track 0.00 -> 48.4 mm
- net RESERVE2: track 0.00 -> 44.9 mm
- net STOP_KEY: track 86.8 -> 45.1 mm
- net RESERVE1: track 0.00 -> 41.6 mm
- net +12V: track 104.2 -> 143.9 mm, vias 2 -> 0
- net BREAK_KEY: track 67.4 -> 29.0 mm
- net +24V: track 90.6 -> 129.0 mm
- net POWER_KEY: track 0.00 -> 29.1 mm
- net POWER_EN_3V3: track 0.00 -> 26.9 mm, vias 0 -> 1
- net MIST_AIR: track 21.9 -> 46.5 mm
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